File: ampli-zero.kicad_pcb (KiCad board)
At the start: 2 copper layers, 100 x 60 mm, 54 parts, among them J1 Conn_01x01, J10 Conn_01x01, J2 Conn_01x01, J3 Conn_01x01, J4 Conn_01x01, J5 Conn_01x01, J6 Conn_01x01, J7 Conn_01x01, J8 Conn_01x01, J9 Conn_01x01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

Commit message: version de 32V
Parts:
- moved R106 0.06 mm to (200.0, 87.8)
Changed lines of the file:
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@@
     (grid_origin 229 101)
     (pcbplotparams
-      (layerselection 0x00010fc_ffffffff)
+      (layerselection 0x0000030_7ffffffe)
       (plot_on_all_layers_selection 0x0000000_00000000)
       (disableapertmacros false)
@@
       (hpglpendiameter 15.000000)
       (dxfpolygonmode true)
-      (dxfimperialunits true)
+      (dxfimperialunits false)
       (dxfusepcbnewfont true)
       (psnegative false)
@@
       (sketchpadsonfab false)
       (subtractmaskfromsilk false)
-      (outputformat 1)
+      (outputformat 3)
       (mirror false)
-      (drillshape 1)
+      (drillshape 0)
       (scaleselection 1)
       (outputdirectory "")
@@
   )
   (footprint "Resistor_THT:R_Axial_Power_L25.0mm_W9.0mm_P27.94mm" (layer "F.Cu")
-    (at 200 87.75 -90)
+    (at 200 87.81 -90)
     (descr "Resistor, Axial_Power series, Box, pin pitch=27.94mm, 7W, length*width*height=25*9*9mm^3, http://cdn-reichelt.de/documents/datenblatt/B400/5WAXIAL_9WAXIAL_11WAXIAL_17WAXIAL%23YAG.pdf")
     (tags "Resistor Axial_Power series Box pin pitch 27.94mm 7W length 25mm width 9mm height 9mm")

Commit message: version que enviada J Angel
Parts:
- added RV1: 5k, Potentiometer_THT:Potentiometer_Runtron_RM-065_Vertical, F.Cu at (169.9, 78.6)
- C3: footprint Capacitor_THT:CP_Radial_D5.0mm_P2.50mm -> Capacitor_THT:CP_Radial_D7.5mm_P2.50mm
- C5: value 300p -> 150p
- C6: footprint Capacitor_THT:CP_Radial_D10.0mm_P5.00mm -> Capacitor_THT:CP_Radial_D12.5mm_P5.00mm
- R23: value 18k -> 91.13k
- moved C6 3.42 mm to (160.5, 116.0)
- moved R101 2.12 mm to (155.5, 78.5)
- moved C3 1.92 mm to (155.5, 83.5)
- moved R115 1.80 mm to (178.4, 87.4)
Connections:
- net +32 renamed +107
- net -32 renamed -107
Routing:
- net /vdt: track 42.8 -> 59.0 mm
- net /vdb: track 56.7 -> 72.0 mm
- net Net-(Q112-B): track 9.34 -> 16.6 mm
- net Net-(J2-Pin_1): track 64.7 -> 61.5 mm
- net -107: track 146.3 -> 143.2 mm
- net Net-(Q102-E): track 4.49 -> 6.61 mm
- net +107: track 128.3 -> 126.2 mm
- net Net-(Q101-E): track 9.40 -> 10.6 mm
- net Net-(J3-Pin_1): track 59.2 -> 59.9 mm
- net /gndv: track 10.3 -> 9.68 mm
- net /VB2: track 36.0 -> 36.6 mm
Other:
- board text added: "0.0000 mm / 0.0000 mm"
- board text added: "0.3000 mm"
- board text added: "1.6000 mm"
- board text added: "100.0000 mm x 60.0000 mm"
- board text added: "2"
- board text added: "BOARD CHARACTERISTICS"
- board text added: "Board Thickness:"
- board text added: "Board overall dimensions:"
- board text added: "Castellated pads:"
- board text added: "Copper Finish:"
- board text added: "Copper Layer Count:"
- board text added: "Edge card connectors:"
- board text added: "Impedance Control:"
- board text added: "Min hole diameter:"
- board text added: "Min track/spacing:"
- board text added: "No"
- board text added: "None"
- board text added: "Plated Board Edge:"

Commit message: agregando potenciometro
Parts:
- R115: value 1.2k -> 1
- R116: value 330 -> 1k
