File: ampli-zero.kicad_sch (KiCad schematic)
At the start: 62 parts, among them J1 Conn_01x01, J10 Conn_01x01, J2 Conn_01x01, J3 Conn_01x01, J4 Conn_01x01, J5 Conn_01x01, J6 Conn_01x01, J7 Conn_01x01, J8 Conn_01x01, J9 Conn_01x01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

Commit message: version de 32V
Parts:
- J1, J10, J2, J3, J4, J5, J6, J7, J8, J9: now left out of the parts list
Other:
- moved on the sheet: C103, L101, L102, R103, R104, R106, R110, R111, R112

Commit message: version que enviada J Angel
Parts:
- added RV1: 5k, Potentiometer_THT:Potentiometer_Runtron_RM-065_Vertical, symbol Device:R_Potentiometer_US
- C3: footprint Capacitor_THT:CP_Radial_D5.0mm_P2.50mm -> Capacitor_THT:CP_Radial_D7.5mm_P2.50mm; VOLTAGE (none) -> 100V
- C5: value 300p -> 150p; VOLTAGE (none) -> >100V
- C6: footprint Capacitor_THT:CP_Radial_D10.0mm_P5.00mm -> Capacitor_THT:CP_Radial_D12.5mm_P5.00mm; V (none) -> 100V
- C7, C8: VOLTAGE (none) -> >100V
- R10, R101, R11, R115, R116, R12, R13, R14, R15, R18, R19, R20, R21, R22, R9: POWER (none) -> 1/2W
- R103, R104: POWER (none) -> 1W
- R23: value 18k -> 91.13k; POWER (none) -> 1/2W
- V1, V2: value 32 -> 107
Connections:
- net vdb: now also RV1.1
- net vdt: now also RV1.3
- net at Q112.2 (B), R115.2, R116.1: now also RV1.2
Other:
- moved on the sheet: C5, C6, R23

Commit message: version desplegada sin probar
Parts:
- removed RV1: 5k, Potentiometer_THT:Potentiometer_Runtron_RM-065_Vertical, symbol Device:R_Potentiometer_US
- R115: value 1.2k -> 1
- R116: value 330 -> 1k
Other:
- note added: "https://audiojudgement.com/"
- note added: "https://circuitdigest.com"
- note added: "https://www.linkedin.com/"
- note removed: "https://audiojudgement.com/speaker-equivalent-circuit/"
- note removed: "https://circuitdigest.com/electronic-circuits/simulate-speaker-with-equivalent-rlc-circuit"
- note removed: "https://www.linkedin.com/pulse/electrical-rlc-model-speaker-parameters-vallabha-hampiholi/"

Commit message: agregando potenciometro
Parts:
- added RV1: 5k, Potentiometer_THT:Potentiometer_Runtron_RM-065_Vertical, symbol Device:R_Potentiometer_US
Connections:
- net vdb: now also RV1.1
- net vdt: now also RV1.3
- net at Q112.2 (B), R115.2, R116.1: now also RV1.2
Changed lines of the file:
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@@
 	)
 	(junction
+		(at 228.6 101.6)
+		(diameter 0)
+		(color 0 0 0 0)
+	)
+	(junction
 		(at 119.38 180.34)
 		(diameter 0)
@@
 	)
 	(junction
+		(at 228.6 173.99)
+		(diameter 0)
+		(color 0 0 0 0)
+	)
+	(junction
 		(at 240.03 110.49)
 		(diameter 0)
@@
 	(wire
 		(pts
-			(xy 217.17 173.99) (xy 232.41 173.99)
+			(xy 217.17 173.99) (xy 228.6 173.99)
 		)
 		(stroke
@@
 	(wire
 		(pts
+			(xy 228.6 173.99) (xy 232.41 173.99)
+		)
+		(stroke
+			(width 0)
+			(type default)
+		)
+	)
+	(wire
+		(pts
 			(xy 140.97 105.41) (xy 140.97 107.95)
 		)
@@
 		)
 	)
+	(wire
+		(pts
+			(xy 217.17 130.81) (xy 224.79 130.81)
+		)
+		(stroke
+			(width 0)
+			(type default)
+		)
+	)
 	(polyline
 		(pts
@@
 	(wire
 		(pts
+			(xy 228.6 134.62) (xy 228.6 173.99)
+		)
+		(stroke
+			(width 0)
+			(type default)
+		)
+	)
+	(wire
+		(pts
 			(xy 119.38 205.74) (xy 119.38 210.82)
 		)
@@
 	(wire
 		(pts
-			(xy 217.17 101.6) (xy 232.41 101.6)
+			(xy 217.17 101.6) (xy 228.6 101.6)
 		)
 		(stroke
@@
 	(wire
 		(pts
+			(xy 228.6 101.6) (xy 228.6 127)
+		)
+		(stroke
+			(width 0)
+			(type default)
+		)
+	)
+	(wire
+		(pts
 			(xy 342.9 139.7) (xy 342.9 142.24)
 		)
@@
 	(wire
 		(pts
+			(xy 228.6 101.6) (xy 232.41 101.6)
+		)
+		(stroke
+			(width 0)
+			(type default)
+		)
+	)
+	(wire
+		(pts
 			(xy 140.97 67.31) (xy 123.19 67.31)
 		)
@@
 					(unit 1)
 				)
+			)
+		)
+	)
+	(symbol
+		(lib_id "Device:R_Potentiometer_US")
+		(at 228.6 130.81 180)
+		(unit 1)
+		(exclude_from_sim no)
+		(in_bom yes)
+		(on_board yes)
+		(dnp no)
+		(fields_autoplaced yes)
+		(property "Reference" "RV1"
+			(at 231.14 129.5399 0)
+			(effects
+				(font
+					(size 1.27 1.27)
+				)
+				(justify right)
+			)
+		)
+		(property "Value" "5k"
+			(at 231.14 132.0799 0)
+			(effects
+				(font
+					(size 1.27 1.27)
+				)
+				(justify right)
+			)
+		)
+		(property "Footprint" "Potentiometer_THT:Potentiometer_Runtron_RM-065_Vertical"
+			(at 228.6 130.81 0)
+			(effects
+				(font
+					(size 1.27 1.27)
+				)
+				(hide yes)
+			)
+		)
+		(property "Datasheet" "~"
+			(at 228.6 130.81 0)
+			(effects
+				(font
+					(size 1.27 1.27)
+				)
+				(hide yes)
+			)
+		)
+		(property "Description" "Potentiometer, US symbol"
+			(at 228.6 130.81 0)
+			(effects
+				(font
+					(size 1.27 1.27)
+				)
+				(hide yes)
+			)
+		)
+		(property "LCSC Part" ""
+			(at 228.6 130.81 0)
+			(effects
+				(font
+					(size 1.27 1.27)
+				)
+				(hide yes)
+			)
+		)
+		(property "Mfr. Part" ""
+			(at 228.6 130.81 0)
+			(effects
+				(font
+					(size 1.27 1.27)
+				)
+				(hide yes)
+			)
+		)
+		(property "Manufacturer" ""
+			(at 228.6 130.81 0)
+			(effects
+				(font
+					(size 1.27 1.27)
+				)
+				(hide yes)
+			)
+		)
+		(property "Price" ""
+			(at 228.6 130.81 0)
+			(effects
+				(font
+					(size 1.27 1.27)
+				)
+				(hide yes)
+			)
+		)
+		(pin "1"
+		)
+		(pin "3"
+		)
+		(pin "2"
+		)
+		(instances
+			(project ""
+				(path "/3cd977d8-8f12-4848-9d60-2993fb1690c7"
+					(reference "RV1")
+					(unit 1)
+				)
